File: Dune/Dune.kicad_pcb (KiCad board)
At the start: 2 copper layers, 278 x 95.9 mm, 90 parts, among them SW1 MK-12C03-G015, SW2 MK-12C03-G015, U1 nice_nano, U2 nice_nano, U3 S2B-PH-K-S(LF)(SN), U4 S2B-PH-K-S(LF)(SN)

Commit message: Add case
Other:
- board size 278 x 95.9 mm -> 278 x 94 mm
Changed lines of the file:
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@@
 	(gr_line
 		(start 177.6495 126.049)
-		(end 162.725 140.95)
+		(end 164.638012 139.04)
 		(stroke
 			(width 0.05)
@@
 	)
 	(gr_line
+		(start 160.633905 139.04)
+		(end 164.637191 139.04)
+		(stroke
+			(width 0.05)
+			(type default)
+		)
+		(layer "Edge.Cuts")
+	)
+	(gr_line
 		(start 177.6495 49.049)
 		(end 177.65 57.65)
@@
 	)
 	(gr_line
-		(start 162.725 140.95)
+		(start 160.635529 139.03488)
 		(end 148.6495 128.049)
 		(stroke
